File: HW6/ME433/ME433.brd (EAGLE design)
At the start: 100 x 80 mm, 43 parts, among them J1 B, J10 HREF, J11 HREF, J12 HREF, J13 HREF, J14 HREF, J15 HREF, J2 A, J3 HREF, J4 PWDN, J5 STR, J6 HREF, J7 HREF, J8 HREF, J9 HREF, U1 PIC32MX170F256B

Commit message: layout
Parts:
- removed LED3: GREEN, ME433:LED3MM
- added J16, J17, J18, J19, J20, J21, J22, J23, J24, J25, J26, J27, J28, J29: (no value), ME433:1X08
- LED2: value RED -> GREEN
- moved J15 343.1 mm to (71.1, 76.2)
- moved J14 339.9 mm to (74.9, 76.2)
- moved J13 336.7 mm to (78.7, 76.2)
- moved J12 300.2 mm to (66.0, 47.0)
- moved J11 297.9 mm to (66.0, 49.5)
- moved J10 295.6 mm to (66.0, 52.1)
- moved J9 293.2 mm to (66.0, 54.6)
- moved J8 290.9 mm to (66.0, 57.1)
- moved J7 288.6 mm to (65.9, 59.7)
- moved J6 286.4 mm to (65.9, 62.4)
- moved J1 277.6 mm to (41.9, 87.6), flipped to the bottom, turned to 90 degrees
- moved R6 272.0 mm to (64.8, 83.8), turned to 180 degrees
- moved J2 264.9 mm to (40.6, 71.1), turned to 90 degrees
- moved U$9 254.4 mm to (64.8, 77.5)
- moved U$10 253.3 mm to (50.8, 76.2)
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Connections:
- new net N$23: J16.8, J17.8, J18.8, J19.8, J20.8
- new net N$24: J16.7, J17.7, J18.7, J19.7, J20.7
- new net N$25: J16.6, J17.6, J18.6, J19.6, J20.6
- new net N$26: J16.5, J17.5, J18.5, J19.5, J20.5
- new net N$27: J16.4, J17.4, J18.4, J19.4, J20.4
- new net N$28: J16.3, J17.3, J18.3, J19.3, J20.3
- new net N$29: J16.2, J17.2, J18.2, J19.2, J20.2
- new net N$30: J16.1, J17.1, J18.1, J19.1, J20.1
- new net N$31: J21.8, J22.8, J23.8, J24.8, J25.8
- new net N$32: J21.7, J22.7, J23.7, J24.7, J25.7
- new net N$33: J21.6, J22.6, J23.6, J24.6, J25.6
- new net N$34: J21.5, J22.5, J23.5, J24.5, J25.5
- new net N$35: J21.4, J22.4, J23.4, J24.4, J25.4
- new net N$36: J21.3, J22.3, J23.3, J24.3, J25.3
- new net N$37: J21.2, J22.2, J23.2, J24.2, J25.2
- new net N$38: J21.1, J22.1, J23.1, J24.1, J25.1
- net +3V3: now also J26.1, J26.2, J26.3, J26.4, J26.5, J26.6, J26.7, J26.8
- net GND: now also J28.1, J28.2, J28.3, J28.4, J28.5, J28.6, J28.7, J28.8, J29.1, J29.2, J29.3, J29.4, J29.5, J29.6, J29.7, J29.8
- net N$3: now also LED2.K; no longer LED3.K
- net N$6: now also LED2.A; no longer LED3.A
- net VIN: now also J27.1, J27.2, J27.3, J27.4, J27.5, J27.6, J27.7, J27.8
Routing:
- net +3V3: track 0.00 -> 298.7 mm, vias 0 -> 3
- net VIN: track 0.00 -> 186.1 mm
- net B15: track 0.00 -> 79.1 mm, vias 0 -> 1
- net B12: track 0.00 -> 76.4 mm, vias 0 -> 1
- net B13: track 0.00 -> 75.0 mm, vias 0 -> 1
- net B14: track 0.00 -> 66.2 mm
- net D2: track 0.00 -> 65.6 mm, vias 0 -> 3
- net WRST: track 0.00 -> 64.8 mm, vias 0 -> 2
- net D0: track 0.00 -> 58.5 mm, vias 0 -> 3
- net D6: track 0.00 -> 56.7 mm
- net B0-PGD-D4: track 0.00 -> 56.7 mm, vias 0 -> 1
- net D1: track 0.00 -> 52.6 mm, vias 0 -> 1
- net B1-PGC-D5: track 0.00 -> 50.0 mm, vias 0 -> 1
- net B7: track 0.00 -> 48.9 mm
- net B6: track 0.00 -> 44.4 mm, vias 0 -> 2
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- added copper zone on layer 16, net GND
Other:
- board size 100 x 80 mm -> 100 x 100 mm
- board text added: "3.3V"
- board text added: "GND"
- board text added: "VIN"
