File: HW6/ME433/ME433.sch (EAGLE design)
At the start: 1 part, among them U1 PIC32MX170F256B

Commit message: schematic
Parts:
- added BAT: (no value), ME433:CONN_02
- added C1, C2, C4: 0.1uF, ME433:C-US025-030X050
- added C3: 10uF, ME433:CPOL-USB45181B
- added J1: B, ME433:CONN_02
- added J10, J11, J12, J13, J14, J15, J3, J6, J7, J8, J9: HREF, ME433:CONN_01
- added J2: A, ME433:CONN_02
- added J4: PWDN, ME433:CONN_01
- added J5: STR, ME433:CONN_01
- added LED1, LED2: RED, ME433:LED3MM
- added LED3: GREEN, ME433:LED3MM
- added R1, R5: 330, ME433:R-US_0207/10
- added R2, R3, R4, R6: 10k, ME433:R-US_0207/10
- added R7, R8: 4.7k, ME433:R-US_0207/10
- added U$1: MICROUSB, ME433:MICROUSB
- added U$10: POLOLUDRV6835, ME433:POLOLUDRV6835
- added U$11: OV7670, ME433:OV7670
- added U$2: SLIDE, ME433:SLIDE
- added U$3: POLOLU3V3, ME433:POLOLU3V3
- added U$4: SNAP, ME433:SNAP
- added U$5: RESET, ME433:PUSH
- added U$6: ADAC2104, ME433:ADAC2104
- added U$7: ST7789, ME433:ST7789
- added U$8: MCP23017, ME433:MCP23017
- added U$9: USER, ME433:PUSH
Connections:
- new net +3V3: C1.1, C2.1, C4.1, LED1.A, R2.2, R3.2, R4.2, R6.2, R7.2, R8.2, U$10.13.VCC, U$10.8.MD, U$11.1.3V3, U$11.13.OE, U$11.8.RST, U$3.1.VOUT, U$4.2.VDD, U$7.2.VCC, U$8.18.RESET, U$8.9.VDD, U1.13.VDD, U1.28.AVDD
- new net +5V: U$1.1.VBUS, U$2.1.VBUS
- new net ADIR: U$10.9.ADIR, U$8.22.A1
- new net APWM: U$10.10.APWM, U$8.23.A2
- new net B0-PGD-D4: U$11.18.D4, U$4.4.PDG, U1.4.B0-PGD
- new net B1-PGC-D5: U$11.5.D5, U$4.5.PGC, U1.5.B1-PGC
- new net B12: U$7.6.DC, U1.23.B12
- new net B13: U$6.2.RXD, U$7.4.SDA, U1.24.B13
- new net B14: U$7.3.SCL, U1.25.B14
- new net B15: U$6.3.TXD, U$7.5.RES, U1.26.B15
- new net B6: R7.1, U$11.2.SIOC, U1.15.B6
- new net B7: R8.1, U$11.21.SIOD, U1.16.B7
- new net B8: R3.1, U$8.12.SCK, U1.17.B8
- new net B9: R4.1, U$8.13.SDA, U1.18.B9
- new net BDIR: U$10.11.DBIR, U$8.24.A3
- new net BPWM: U$10.12.BPWM, U$8.25.A4
- new net D0: U$11.16.D0, U1.2.A0
- new net D1: U$11.7.D1, U1.3.A1
- new net D2: U$11.17.D2, U1.9.A2
- new net D3: U$11.6.D3, U1.10.A3
- new net D6: U$11.19.D6, U1.6.B2
- new net D7: U$11.4.D7, U1.7.B3
- new net GND: BAT.1, C1.2, C2.2, C3.-, C4.2, R1.1, R5.1, U$1.5.GND, U$10.1.GND, U$10.14.GND, U$11.22.GND, U$3.2.GND, U$4.3.GND, U$5.1, U$6.6.GND, U$7.1.GND, U$8.10.VSS, U$8.15.AD0, U$8.16.AD1, U$8.17.AD2, U$9.1, U1.19.VSS, U1.27.AVSS, U1.8.VSS
- new net MCLR: R2.1, U$4.1.MCLR, U$5.2, U1.1.MCLR
- new net N$1: LED1.C, R1.2
- new net N$10: J5.1, U$11.9.STR
- new net N$11: J4.1, U$11.15.PWDN
- new net N$12: J3.1, U$11.20.HREF
- new net N$13: J6.1, U$8.2.B1
- new net N$14: J7.1, U$8.3.B2
- new net N$15: J8.1, U$8.4.B3
- new net N$16: J9.1, U$8.5.B4
- new net N$17: J10.1, U$8.6.B5
- new net N$18: J11.1, U$8.7.B6
- new net N$19: J12.1, U$8.8.B7
- new net N$2: C3.+, U1.20.VCAP
- new net N$20: J13.1, U$8.28.A7
- new net N$21: J14.1, U$8.27.A6
- new net N$22: J15.1, U$8.26.A5
- new net N$3: LED3.C, R5.2
- new net N$4: J1.2, U$10.3.BO2
- new net N$5: J1.1, U$10.4.BO1
- new net N$6: LED3.A, U$8.21.A0
- new net N$7: R6.1, U$8.1.B0, U$9.2
- new net N$8: J2.2, U$10.5.AO2
- new net N$9: J2.1, U$10.6.AO1
- new net RCK: U$11.14.RCK, U1.12.A4
- new net RRST: U$11.12.RRST, U1.21.B10
- new net V+: BAT.2, U$2.3.VBAT
- new net VIN: U$10.2.VIN, U$2.2.VOUT, U$3.3.VIN
- new net VSY: U$11.3.VSY, U1.11.B4
- new net WR: U$11.10.WR, U1.14.B5
- new net WRST: U$11.11.WRST, U1.22.B11
Other:
- note added: "B12 - DC"
- note added: "B13 - U1RX, SDO1"
- note added: "B14 - SCK1"
- note added: "B15 - U1TX, RES"
- note added: "B6 - SIOC"
- note added: "B7 - SIOD"
- note added: "B8 - SCL1"
- note added: "B9 - SDA1"
- moved on the sheet: U1

Commit message: layout
Parts:
- removed LED3: GREEN, ME433:LED3MM
- added J16, J17, J18, J19, J20, J21, J22, J23, J24, J25, J26, J27, J28, J29: (no value), ME433:CONN_08"
- LED2: value RED -> GREEN
Connections:
- new net N$23: J16.8, J17.8, J18.8, J19.8, J20.8
- new net N$24: J16.7, J17.7, J18.7, J19.7, J20.7
- new net N$25: J16.6, J17.6, J18.6, J19.6, J20.6
- new net N$26: J16.5, J17.5, J18.5, J19.5, J20.5
- new net N$27: J16.4, J17.4, J18.4, J19.4, J20.4
- new net N$28: J16.3, J17.3, J18.3, J19.3, J20.3
- new net N$29: J16.2, J17.2, J18.2, J19.2, J20.2
- new net N$30: J16.1, J17.1, J18.1, J19.1, J20.1
- new net N$31: J21.8, J22.8, J23.8, J24.8, J25.8
- new net N$32: J21.7, J22.7, J23.7, J24.7, J25.7
- new net N$33: J21.6, J22.6, J23.6, J24.6, J25.6
- new net N$34: J21.5, J22.5, J23.5, J24.5, J25.5
- new net N$35: J21.4, J22.4, J23.4, J24.4, J25.4
- new net N$36: J21.3, J22.3, J23.3, J24.3, J25.3
- new net N$37: J21.2, J22.2, J23.2, J24.2, J25.2
- new net N$38: J21.1, J22.1, J23.1, J24.1, J25.1
- net +3V3: now also J26.1, J26.2, J26.3, J26.4, J26.5, J26.6, J26.7, J26.8
- net GND: now also J28.1, J28.2, J28.3, J28.4, J28.5, J28.6, J28.7, J28.8, J29.1, J29.2, J29.3, J29.4, J29.5, J29.6, J29.7, J29.8
- net N$3: now also LED2.C; no longer LED3.C
- net N$6: now also LED2.A; no longer LED3.A
- net VIN: now also J27.1, J27.2, J27.3, J27.4, J27.5, J27.6, J27.7, J27.8
Other:
- moved on the sheet: LED2
